Commit message: fix: 1002新建moveit包 解决机器状态不变问题

File: innfos_control/gazebo_control/models/arm.urdf.xacro (robot description, xacro)
@@ -15,5 +15,5 @@
 </xacro:macro>
 <link
-    name="${prefix}_base_link">
+    name="base_link">
     <inertial>
       <origin
@@ -85,5 +85,5 @@
       rpy="3.4694E-18 2.4378E-13 -3.1416" />
     <parent
-      link="${prefix}_base_link" />
+      link="base_link" />
     <child
       link="link1" />

File: innfos_control/gazebo_control/models/turtle.urdf.xacro (robot description, xacro)
@@ -7,8 +7,8 @@
   <joint name="base_joint" type="fixed">
     <parent link="base_footprint"/>
-    <child link="base_link" />
+    <child link="turtle_base_link" />
     <origin xyz="0 0 0.010" rpy="0 0 0"/>
   </joint>
-  <link name="base_link">
+  <link name="turtle_base_link">
     <visual>
       <origin xyz="-0.064 0 0.0" rpy="0 0 0"/>
@@ -31,5 +31,5 @@
   </link>
   <joint name="wheel_left_joint" type="continuous">
-    <parent link="base_link"/>
+    <parent link="turtle_base_link"/>
     <child link="wheel_left_link"/>
     <origin xyz="0.0 0.144 0.023" rpy="-1.57 0 0"/>
@@ -59,5 +59,5 @@
   </link>
   <joint name="wheel_right_joint" type="continuous">
-    <parent link="base_link"/>
+    <parent link="turtle_base_link"/>
     <child link="wheel_right_link"/>
     <origin xyz="0.0 -0.144 0.023" rpy="-1.57 0 0"/>
@@ -87,5 +87,5 @@
   </link>
   <joint name="caster_back_right_joint" type="fixed">
-    <parent link="base_link"/>
+    <parent link="turtle_base_link"/>
     <child link="caster_back_right_link"/>
     <origin xyz="-0.177 -0.064 -0.004" rpy="-1.57 0 0"/>
@@ -107,5 +107,5 @@
   </link>
   <joint name="caster_back_left_joint" type="fixed">
-    <parent link="base_link"/>
+    <parent link="turtle_base_link"/>
     <child link="caster_back_left_link"/>
     <origin xyz="-0.177 0.064 -0.004" rpy="-1.57 0 0"/>
@@ -127,5 +127,5 @@
   </link>
   <joint name="imu_joint" type="fixed">
-    <parent link="base_link"/>
+    <parent link="turtle_base_link"/>
     <child link="imu_link"/>
     <origin xyz="0.0 0 0.068" rpy="0 0 0"/>
@@ -133,5 +133,5 @@
   <link name="imu_link"/>
   <joint name="scan_joint" type="fixed">
-    <parent link="base_link"/>
+    <parent link="turtle_base_link"/>
     <child link="base_scan"/>
     <origin xyz="-0.064 0 0.122" rpy="0 0 0"/>
@@ -161,5 +161,5 @@
   <joint name="camera_joint" type="fixed">
     <origin xyz="0.073 -0.011 0.084" rpy="0 0 0"/>
-    <parent link="base_link"/>
+    <parent link="turtle_base_link"/>
     <child link="camera_link"/>
   </joint>

File: innfos_control/gazebo_control/models/yang.urdf.xacro (robot description, xacro)
@@ -7,5 +7,5 @@
 <joint name="connent_joint" type="fixed">
     <parent link="base_footprint" />
-    <child link="arm_base_link" />
+    <child link="base_link" />
     <origin xyz="-0.05 0.0 0.2" rpy="0.0 0.0 0" />
 </joint>
